File: hardware/PD_Micro.kicad_pcb (KiCad board)
At the start: 4 copper layers, 40.6 x 17.8 mm, 61 parts, among them J1 Conn_01x02, J2 Conn_01x02, J3 Conn_01x02, J4 Conn_01x12, J5 Conn_01x12, Q1 DMP3017SFK, Q2 DTC143E, SW1 SW_Push, U1 TPS62175DQC, U2 SRV05-4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

Commit message: update
Other:
- net class Default removed
- net class Minimum removed
